File: ESP8266-Breakout/ESP8266-Breakout.sch (KiCad schematic (older format))
At the start: 9 parts, among them J101 Conn_01x09_Female, J102 Conn_01x09_Female, U101 AMS1117-3.3

Commit message: Single and panel board views added
Parts:
- C101, C104: LCSC C96123 -> C13585
- C102, C103: LCSC C96123 -> C24497
Changed lines of the file:
@@
 F 4 "10V" H 3250 6700 50  0001 C CNN "Maximum Value"
 F 5 "1206" H 3250 6700 50  0001 C CNN "Package Reference"
-F 6 "C96123" H 3250 6700 50  0001 C CNN "LCSC"
+F 6 "C13585" H 3250 6700 50  0001 C CNN "LCSC"
 	1    3250 6700
 	1    0    0    -1
@@
 F 4 "10V" H 2900 6700 50  0001 C CNN "Maximum Value"
 F 5 "1206" H 2900 6700 50  0001 C CNN "Package Reference"
-F 6 "C96123" H 2900 6700 50  0001 C CNN "LCSC"
+F 6 "C24497" H 2900 6700 50  0001 C CNN "LCSC"
 	1    2900 6700
 	1    0    0    -1
@@
 F 4 "10V" H 2000 6700 50  0001 C CNN "Maximum Value"
 F 5 "1206" H 2000 6700 50  0001 C CNN "Package Reference"
-F 6 "C96123" H 2000 6700 50  0001 C CNN "LCSC"
+F 6 "C24497" H 2000 6700 50  0001 C CNN "LCSC"
 	1    2000 6700
 	1    0    0    -1
@@
 F 4 "10V" H 1700 6700 50  0001 C CNN "Maximum Value"
 F 5 "1206" H 1700 6700 50  0001 C CNN "Package Reference"
-F 6 "C96123" H 1700 6700 50  0001 C CNN "LCSC"
+F 6 "C13585" H 1700 6700 50  0001 C CNN "LCSC"
 	1    1700 6700
 	1    0    0    -1
