File: ESP8266-Breakout/ESP8266.sch (KiCad schematic (older format))
At the start: 16 parts, among them J501 FTDI, SW501 Flash, SW502 RST, U501 ESP-12F

Commit message: Single and panel board views added
Parts:
- SW501, SW502: LCSC C319365 -> C398053; LCSC (alt) C398053 -> C354943
Changed lines of the file:
@@
 F 2 "Button_Switch_SMD:SW_SPST_CK_RS282G05A3" H 1650 5550 50  0001 C CNN
 F 3 "~" H 1650 5550 50  0001 C CNN
-F 4 "C319365" H 1650 5350 50  0001 C CNN "LCSC"
+F 4 "C398053" H 1650 5350 50  0001 C CNN "LCSC"
 F 5 "" H 1650 5350 50  0001 C CNN "Maximum Value"
 F 6 "6.1x3.7x2.5mm" H 1650 5350 50  0001 C CNN "Package Reference"
-F 7 "C398053" V 1650 5350 50  0001 C CNN "LCSC (alt)"
+F 7 "C354943" V 1650 5350 50  0001 C CNN "LCSC (alt)"
 	1    1650 5350
 	0    -1   -1   0
@@
 F 2 "Button_Switch_SMD:SW_SPST_CK_RS282G05A3" H 4050 5450 50  0001 C CNN
 F 3 "~" H 4050 5450 50  0001 C CNN
-F 4 "C319365" H 4050 5250 50  0001 C CNN "LCSC"
+F 4 "C398053" H 4050 5250 50  0001 C CNN "LCSC"
 F 5 "" H 4050 5250 50  0001 C CNN "Maximum Value"
 F 6 "6.1x3.7x2.5mm" H 4050 5250 50  0001 C CNN "Package Reference"
-F 7 "C398053" V 4050 5250 50  0001 C CNN "LCSC (alt)"
+F 7 "C354943" V 4050 5250 50  0001 C CNN "LCSC (alt)"
 	1    4050 5250
 	0    -1   -1   0
